File: PCB_Design/Kicad_Workspace/MCU Embedded PCB_AT2/STM32F103x8/STM32F103x8.kicad_sch (KiCad schematic)
At the start: 16 parts, among them J1 Conn_01x17, J2 Conn_01x05, J3 Conn_01x01, J4 USB_A, J5 Conn_01x04, J6 Conn_01x08, SW1 SW_Push, U1 STM32F103C8Tx, U2 AP2204R-3.3, Y1 8MHz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

Commit message: update_stm
Parts:
- removed C5: C, Capacitor_THT:C_Axial_L3.8mm_D2.6mm_P7.50mm_Horizontal, symbol Device:C
- SW1: footprint Button_Switch_THT:SW_PUSH-12mm -> Button_Switch_THT:SW_PUSH_1P1T_6x3.5mm_H4.3_APEM_MJTP1243
Connections:
- net GND: now also J4.5 (Shield)
- no-connect marks 4 -> 3
Other:
- moved on the sheet: C2, SW1, U2, Y2

Commit message: update_stm
Parts:
- Y2: footprint Oscillator:Oscillator_SMD_TXC_7C-4Pin_5.0x3.2mm_HandSoldering -> Crystal:Crystal_SMD_Abracon_ABM3-2Pin_5.0x3.2mm
Changed lines of the file:
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@@
 			)
 		)
-		(property "Footprint" "Oscillator:Oscillator_SMD_TXC_7C-4Pin_5.0x3.2mm_HandSoldering"
+		(property "Footprint" "Crystal:Crystal_SMD_Abracon_ABM3-2Pin_5.0x3.2mm"
 			(at 189.23 78.74 0)
 			(effects
